Commit message: URDFとSDFが一致するようにし，表記を整理

File: turtlebot3_description/urdf/turtlebot3_happy_mini.urdf (robot description, URDF)
Before this commit: robot turtlebot3_happy_mini, 11 links, 10 joints
Links:
- removed link camera_rgb_frame
- removed link caster_back_left_link
- removed link caster_back_right_link
- added link caster_back_link, mass 0.001; collision sphere radius=0.005
- added link caster_front_link, mass 0.001; collision sphere radius=0.005
- link base_link: geometry collision cylinder length=1.1 radius=0.18; visual mesh filename=package://turtlebot3_description/meshes/happy_mini/arm_mini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 scale=0.01 0.01 0.01
- link base_scan: geometry collision box size=0.06 0.06 0.087; visual mesh filename=package://turtlebot3_description/meshes/happy_mini/lidar.dae scale=1 1 1
- link camera_link: mass None -> 0.035; geometry collision box size=0.04 0.18 0.025
Joints:
- removed joint camera_rgb_optical_joint
- removed joint caster_back_left_joint
- removed joint caster_back_right_joint
- added joint caster_back_joint: type fixed, parent base_link, child caster_back_link, origin xyz=-0.144 0.0 -0.004 rpy=0 0 0
- added joint caster_front_joint: type fixed, parent base_link, child caster_front_link, origin xyz=0.144 0.0 -0.004 rpy=0 0 0
- joint camera_joint: origin xyz=0.073 -0.011 0.084 rpy=0 0 0 -> xyz=0.08 0 1.03 rpy=0 0 0
- joint camera_rgb_joint: child camera_rgb_frame -> camera_rgb_optical_frame; origin xyz=0.003 0.011 0.009 rpy=0 0 0 -> xyz=0.0 0.0 0.0 rpy=-1.57 0 -1.57
- joint imu_joint: origin xyz=0.0 0 0.068 rpy=0 0 0 -> xyz=-0.032 0 0.068 rpy=0 0 0
- joint scan_joint: origin xyz=-0.064 0 0.122 rpy=0 0 0 -> xyz=0.14 0 0.121 rpy=0 0 0
